Commit message: urdf硬件接口控制器

File: src/robot/urdf/hardware.xacro (robot description, xacro)
@@ -1,98 +1,73 @@
 <?xml version="1.0"?>
-<robot xmlns:xacro="http://www.ros.org/wiki/xacro">
-  <!--
-    硬件接口配置
-    定义所有可控制的关节及其命令/状态接口
-    如果需要参数化（例如关节名称列表），可以使用 xacro 属性传递
-  -->
-  <ros2_control name="robot_control" type="system">
+<robot name="robot_hardware" xmlns:xacro="http://www.ros.org/wiki/xacro">
+  <ros2_control name="RobotHardware" type="system">
     <hardware>
-      <!-- 根据仿真环境选择插件：fake_components 用于测试，gazebo 用于仿真 -->
-      <plugin>fake_components/GenericSystem</plugin>
-      <!-- 列出所有受控关节，确保与下文定义一致 -->
-      <param name="joints">lap_body_joint_rf lap_body_joint_lf lap_body_joint_rr lap_body_joint_lr shin_lap_rf_joint_rf shin_lap_lf_joint_lf shin_lap_rr_joint_rr shin_lap_lr_joint_lr motor_shin_rf_joint_rf motor_shin_lf_joint_lf motor_shin_rr_joint_rr motor_shin_lr_joint_lr wheel_motor_rf_joint_rf wheel_motor_lf_joint_lf wheel_motor_rr_joint_rr wheel_motor_lr_joint_lr</param>
+      <!-- 🔥 官方自带插件，无需安装任何依赖！ -->
+      <plugin>mock_components/GenericSystem</plugin>
     </hardware>
-    <!-- 大腿关节 -->
-    <joint name="lap_body_joint_rf">
+    <joint name="lap_body_joint_fr">
       <command_interface name="position"/>
       <state_interface name="position"/>
-      <state_interface name="velocity"/>
     </joint>
-    <joint name="lap_body_joint_lf">
+    <joint name="lap_body_joint_fl">
       <command_interface name="position"/>
       <state_interface name="position"/>
-      <state_interface name="velocity"/>
     </joint>
     <joint name="lap_body_joint_rr">
       <command_interface name="position"/>
       <state_interface name="position"/>
-      <state_interface name="velocity"/>
     </joint>
-    <joint name="lap_body_joint_lr">
+    <joint name="lap_body_joint_rl">
       <command_interface name="position"/>
       <state_interface name="position"/>
-      <state_interface name="velocity"/>
     </joint>
-    <!-- 小腿关节 -->
-    <joint name="shin_lap_rf_joint_rf">
+    <joint name="shin_lap_fr_joint_fr">
       <command_interface name="position"/>
       <state_interface name="position"/>
-      <state_interface name="velocity"/>
     </joint>
-    <joint name="shin_lap_lf_joint_lf">
+    <joint name="shin_lap_fl_joint_fl">
       <command_interface name="position"/>
       <state_interface name="position"/>
-      <state_interface name="velocity"/>
     </joint>
     <joint name="shin_lap_rr_joint_rr">
       <command_interface name="position"/>
       <state_interface name="position"/>
+    </joint>
+    <joint name="shin_lap_rl_joint_rl">
+      <command_interface name="position"/>
+      <state_interface name="position"/>
+    </joint>
+    <!-- 转向关节（和你的 motor.xacro 完全匹配） -->
+    <joint name="front_right_steer_joint">
+      <command_interface name="position"/>
+      <state_interface name="position"/>
+    </joint>
+    <joint name="front_left_steer_joint">
+      <command_interface name="position"/>
+      <state_interface name="position"/>
+    </joint>
+    <joint name="rear_right_steer_joint">
+      <command_interface name="position"/>
+      <state_interface name="position"/>
+    </joint>
+    <joint name="rear_left_steer_joint">
+      <command_interface name="position"/>
+      <state_interface name="position"/>
+    </joint>
+    <!-- 轮子关节（和你的 wheel.xacro 完全匹配） -->
+    <joint name="front_right_wheel_joint">
+      <command_interface name="velocity"/>
       <state_interface name="velocity"/>
     </joint>
-    <joint name="shin_lap_lr_joint_lr">
-      <command_interface name="position"/>
-      <state_interface name="position"/>
+    <joint name="front_left_wheel_joint">
+      <command_interface name="velocity"/>
       <state_interface name="velocity"/>
     </joint>
-    <!-- 转向电机关节 -->
-    <joint name="motor_shin_rf_joint_rf">
-      <command_interface name="position"/>
-      <state_interface name="position"/>
+    <joint name="rear_right_wheel_joint">
+      <command_interface name="velocity"/>
       <state_interface name="velocity"/>
     </joint>
-    <joint name="motor_shin_lf_joint_lf">
-      <command_interface name="position"/>
-      <state_interface name="position"/>
-      <state_interface name="velocity"/>
-    </joint>
-    <joint name="motor_shin_rr_joint_rr">
-      <command_interface name="position"/>
-      <state_interface name="position"/>
-      <state_interface name="velocity"/>
-    </joint>
-    <joint name="motor_shin_lr_joint_lr">
-      <command_interface name="position"/>
-      <state_interface name="position"/>
-      <state_interface name="velocity"/>
-    </joint>
-    <!-- 轮子关节（速度控制） -->
-    <joint name="wheel_motor_rf_joint_rf">
+    <joint name="rear_left_wheel_joint">
       <command_interface name="velocity"/>
-      <state_interface name="position"/>
-      <state_interface name="velocity"/>
-    </joint>
-    <joint name="wheel_motor_lf_joint_lf">
-      <command_interface name="velocity"/>
-      <state_interface name="position"/>
-      <state_interface name="velocity"/>
-    </joint>
-    <joint name="wheel_motor_rr_joint_rr">
-      <command_interface name="velocity"/>
-      <state_interface name="position"/>
-      <state_interface name="velocity"/>
-    </joint>
-    <joint name="wheel_motor_lr_joint_lr">
-      <command_interface name="velocity"/>
-      <state_interface name="position"/>
       <state_interface name="velocity"/>
     </joint>

File: src/robot/urdf/lap.xacro (robot description, xacro)
@@ -13,5 +13,5 @@
         <origin xyz="0 0 0" rpy="0 0 0"/>
         <geometry>
-          <mesh filename="package://robot/meshes/lap-rf.obj"
+          <mesh filename="${mesh_path}/lap-rf.obj"
                 scale="${mesh_scale}"/>
         </geometry>
@@ -22,5 +22,5 @@
         <origin xyz="0 0 0" rpy="0 0 0"/>
         <geometry>
-          <mesh filename="package://robot/meshes/lap-rf.obj"
+          <mesh filename="${mesh_path}/lap-rf.obj"
                 scale="${mesh_scale}"/>
         </geometry>

File: src/robot/urdf/motor.xacro (robot description, xacro)
@@ -11,5 +11,5 @@
   -->
   <xacro:macro name="motor"
-               params="suffix parent_link
+               params="suffix parent_link joint_position
                        xyz:='0 0 0'
                        rpy:='0 0 0'
@@ -20,5 +20,5 @@
         <origin xyz="0 0 0" rpy="0 0 0"/>
         <geometry>
-          <mesh filename="package://robot/meshes/motor-rf.obj"
+          <mesh filename="${mesh_path}/motor-rf.obj"
                 scale="${mesh_scale}"/>
         </geometry>
@@ -29,5 +29,5 @@
         <origin xyz="0 0 0" rpy="0 0 0"/>
         <geometry>
-          <mesh filename="package://robot/meshes/motor-rf.obj"
+          <mesh filename="${mesh_path}/motor-rf.obj"
                 scale="${mesh_scale}"/>
         </geometry>
@@ -42,5 +42,5 @@
     </link>
     <!-- 转向关节（绕 Z 轴旋转，左右各 90 度） -->
-    <joint name="motor_${parent_link}_joint_${suffix}" type="revolute">
+    <joint name="${joint_position}_steer_joint" type="revolute">
       <origin xyz="${xyz}" rpy="${rpy}"/>
       <parent link="${parent_link}"/>

File: src/robot/urdf/robot.xacro (robot description, xacro)
@@ -7,4 +7,11 @@
   <xacro:include filename="motor.xacro"/>
   <xacro:include filename="wheel.xacro"/>
+  <xacro:include filename="radar-front.xacro"/>
+  <xacro:include filename="radar-side.xacro"/>
+  <xacro:include filename="imu.xacro"/>
+  <!-- 新增：动态获取robot包的绝对路径（核心！） -->
+  <xacro:property name="pkg_path" value="$(find robot)"/>
+  <!-- 定义mesh文件夹路径 -->
+  <xacro:property name="mesh_path" value="${pkg_path}/meshes"/>
   <!-- 基础连杆（作为机器人根节点） -->
   <link name="base_link">
@@ -15,7 +22,5 @@
         <box size="0 0 0"/> <!-- 小方块作为base_link可视化 -->
       </geometry>
-      <material name="red">
-        <diffuse>1 0 0 1</diffuse>
-      </material>
+      <xacro:get_material_by_name material_name="pla_gray_light"/>
     </visual>
   </link>
@@ -26,5 +31,5 @@
       <origin xyz="0 0 0" rpy="0 0 0"/>
       <geometry>
-        <mesh filename="package://robot/meshes/body.obj"
+        <mesh filename="${mesh_path}/body.obj"
               scale="0.001 0.001 0.001"/>
       </geometry>
@@ -35,5 +40,5 @@
       <origin xyz="0 0 0" rpy="0 0 0"/>
       <geometry>
-        <mesh filename="package://robot/meshes/body.obj"
+        <mesh filename="${mesh_path}/body.obj"
               scale="0.001 0.001 0.001"/>
       </geometry>
@@ -56,5 +61,5 @@
   <!-- 大腿部分（保留所有lap宏调用，确保关节可被GUI控制） -->
   <!-- 右前大腿 - 原样 -->
-  <xacro:lap suffix="rf"
+  <xacro:lap suffix="fr"
              parent_link="body"
              xyz="-0.091 -0.072 0.158"
@@ -62,5 +67,5 @@
              mesh_scale="0.001 0.001 0.001"/>
   <!-- 左前大腿 - Y轴镜像 -->
-  <xacro:lap suffix="lf"
+  <xacro:lap suffix="fl"
              parent_link="body"
              xyz="0.091 -0.072 0.158"
@@ -74,5 +79,5 @@
              mesh_scale="0.001 -0.001 0.001"/> <!-- X轴镜像 -->
   <!-- 左后大腿 - X和Y轴都镜像 -->
-  <xacro:lap suffix="lr"
+  <xacro:lap suffix="rl"
              parent_link="body"
              xyz="0.091 0.072 0.158"
@@ -81,12 +86,12 @@
   <!-- 小腿部分 -->
   <!-- 右前小腿 -->
-  <xacro:shin suffix="rf"
-              parent_link="lap_rf"
+  <xacro:shin suffix="fr"
+              parent_link="lap_fr"
               xyz="-0.017 -0.060 0"
               rpy="0 0 0"
               mesh_scale="0.001 0.001 0.001"/>
   <!-- 左前小腿（Y轴镜像） -->
-  <xacro:shin suffix="lf"
-              parent_link="lap_lf"
+  <xacro:shin suffix="fl"
+              parent_link="lap_fl"
               xyz="0.017 -0.060 0"
               rpy="0 0 0"
@@ -99,17 +104,19 @@
               mesh_scale="0.001 -0.001 0.001"/>
   <!-- 左后小腿（X和Y轴镜像） -->
-  <xacro:shin suffix="lr"
-              parent_link="lap_lr"
+  <xacro:shin suffix="rl"
+              parent_link="lap_rl"
               xyz="0.017 0.060 0"
               rpy="0 0 0"
               mesh_scale="-0.001 -0.001 0.001"/>
   <!-- 转向部分 -->
-  <xacro:motor suffix="rf"
-              parent_link="shin_rf"
+  <xacro:motor suffix="fr"
+              parent_link="shin_fr"
+              joint_position="front_right"
               xyz="-0.008 0 -0.069"
               rpy="0 0 0"
               mesh_scale="0.001 0.001 0.001"/>
-  <xacro:motor suffix="lf"
-              parent_link="shin_lf"
+  <xacro:motor suffix="fl"
+              parent_link="shin_fl"
+              joint_position="front_left"
               xyz="0.008 0 -0.069"
               rpy="0 0 0"
@@ -117,20 +124,24 @@
   <xacro:motor suffix="rr"
               parent_link="shin_rr"
+              joint_position="rear_right"
               xyz="-0.008 0 -0.069"
               rpy="0 0 0"
               mesh_scale="0.001 -0.001 0.001"/>
-  <xacro:motor suffix="lr"
-              parent_link="shin_lr"
+  <xacro:motor suffix="rl"
+              parent_link="shin_rl"
+              joint_position="rear_left"
               xyz="0.008 0 -0.069"
               rpy="0 0 0"
               mesh_scale="-0.001 -0.001 0.001"/>
   <!-- 轮胎部分-->
-  <xacro:wheel suffix="rf"
-             parent_link="motor_rf"
+  <xacro:wheel suffix="fr"
+             parent_link="motor_fr"
+             joint_position="front_right"
              xyz="0.015 0 -0.085"
              rpy="0 0 0"
              mesh_scale="0.001 0.001 0.001"/>
-  <xacro:wheel suffix="lf"
-             parent_link="motor_lf"
+  <xacro:wheel suffix="fl"
+             parent_link="motor_fl"
+             joint_position="front_left"
              xyz="-0.015 0 -0.085"
              rpy="0 0 0"
@@ -138,16 +149,66 @@
   <xacro:wheel suffix="rr"
              parent_link="motor_rr"
+             joint_position="rear_right"
              xyz="0.015 0 -0.085"
              rpy="0 0 0"
              mesh_scale="0.001 -0.001 0.001"/>
-  <xacro:wheel suffix="lr"
-             parent_link="motor_lr"
+  <xacro:wheel suffix="rl"
+             parent_link="motor_rl"
+             joint_position="rear_left"
              xyz="-0.015 0 -0.085"
              rpy="0 0 0"
              mesh_scale="-0.001 -0.001 0.001"/>
+  <!-- 前超声波传感器-->
+  <xacro:radar-front suffix="fr"
+              parent_link="motor_fr"
+              xyz="0 -0.037 -0.011"
+              rpy="0 0 0"
+              mesh_scale="0.001 0.001 0.001"/>
+  <xacro:radar-front suffix="fl"
+              parent_link="motor_fl"
+              xyz="0 -0.037 -0.011"
+              rpy="0 0 0"
+              mesh_scale="-0.001 0.001 0.001"/>
+  <xacro:radar-front suffix="rr"
+              parent_link="motor_rr"
+              xyz="0 0.037 -0.011"
+              rpy="0 0 0"
+              mesh_scale="0.001 -0.001 0.001"/>
+  <xacro:radar-front suffix="rl"
+              parent_link="motor_rl"
+              xyz="0 0.037 -0.011"
+              rpy="0 0 0"
+              mesh_scale="-0.001 -0.001 0.001"/>
+  <!-- 侧超声波传感器-->
+  <xacro:radar-side suffix="fr"
+              parent_link="shin_fr"
+              xyz="-0.026 -0.009 -0.035"
+              rpy="0 0 0"
+              mesh_scale="0.001 0.001 0.001"/>
+  <xacro:radar-side suffix="fl"
+              parent_link="shin_fl"
+              xyz="0.026 -0.009 -0.035"
+              rpy="0 0 0"
+              mesh_scale="-0.001 0.001 0.001"/>
+  <xacro:radar-side suffix="rr"
+              parent_link="shin_rr"
+              xyz="-0.026 0.009 -0.035"
+              rpy="0 0 0"
+              mesh_scale="0.001 -0.001 0.001"/>
+  <xacro:radar-side suffix="rl"
+              parent_link="shin_rl"
+              xyz="0.026 0.009 -0.035"
+              rpy="0 0 0"
+              mesh_scale="-0.001 -0.001 0.001"/>
+  <!--  插入 IMU（修改安装位置即可） -->
+  <xacro:imu
+    parent_link="body"
+    x="0.0"
+    y="0.0"
+    z="0.15"
+    roll="0"
+    pitch="0"
+    yaw="0"
+  />
   <xacro:include filename="hardware.xacro"/>
-  <!-- 移除所有ros2_control和Gazebo相关配置 -->
-  <!-- 1. 移除ros2_control硬件接口配置 -->
-  <!-- 2. 移除gazebo插件配置 -->
-  <!-- 3. 移除所有gazebo标签下的材质/物理属性配置 -->
 </robot>

File: src/robot/urdf/shin.xacro (robot description, xacro)
@@ -20,5 +20,5 @@
         <origin xyz="0 0 0" rpy="0 0 0"/>
         <geometry>
-          <mesh filename="package://robot/meshes/shin-rf.obj"
+          <mesh filename="${mesh_path}/shin-rf.obj"
                 scale="${mesh_scale}"/>
         </geometry>
@@ -28,5 +28,5 @@
         <origin xyz="0 0 0" rpy="0 0 0"/>
         <geometry>
-          <mesh filename="package://robot/meshes/shin-rf.obj"
+          <mesh filename="${mesh_path}/shin-rf.obj"
                 scale="${mesh_scale}"/>
         </geometry>

File: src/robot/urdf/wheel.xacro (robot description, xacro)
@@ -11,5 +11,5 @@
   -->
   <xacro:macro name="wheel"
-               params="suffix parent_link
+               params="suffix parent_link joint_position
                        xyz:='0 0 0'
                        rpy:='0 0 0'
@@ -20,5 +20,5 @@
         <origin xyz="0 0 0" rpy="0 0 0"/>
         <geometry>
-          <mesh filename="package://robot/meshes/wheel-rf.obj"
+          <mesh filename="${mesh_path}/wheel-rf.obj"
                 scale="${mesh_scale}"/>
         </geometry>
@@ -29,5 +29,5 @@
         <origin xyz="0 0 0" rpy="0 0 0"/>
         <geometry>
-          <mesh filename="package://robot/meshes/wheel-rf.obj"
+          <mesh filename="${mesh_path}/wheel-rf.obj"
                 scale="${mesh_scale}"/>
         </geometry>
@@ -43,5 +43,5 @@
     </link>
     <!-- 轮子旋转关节（连续旋转） -->
-    <joint name="wheel_${parent_link}_joint_${suffix}" type="continuous">
+    <joint name="${joint_position}_wheel_joint" type="continuous">
       <origin xyz="${xyz}" rpy="${rpy}"/>
       <parent link="${parent_link}"/>

Commit message: urdf修改

File: src/robot/urdf/hardware.xacro (robot description, xacro)
@@ -58,16 +58,20 @@
     <joint name="front_right_wheel_joint">
       <command_interface name="velocity"/>
+      <state_interface name="position"/>
       <state_interface name="velocity"/>
     </joint>
     <joint name="front_left_wheel_joint">
       <command_interface name="velocity"/>
+      <state_interface name="position"/>
       <state_interface name="velocity"/>
     </joint>
     <joint name="rear_right_wheel_joint">
       <command_interface name="velocity"/>
+      <state_interface name="position"/>
       <state_interface name="velocity"/>
     </joint>
     <joint name="rear_left_wheel_joint">
       <command_interface name="velocity"/>
+      <state_interface name="position"/>
       <state_interface name="velocity"/>
     </joint>

File: src/robot/urdf/lap.xacro (robot description, xacro)
@@ -13,5 +13,5 @@
         <origin xyz="0 0 0" rpy="0 0 0"/>
         <geometry>
-          <mesh filename="${mesh_path}/lap-rf.obj"
+          <mesh filename="package://robot/meshes/lap-rf.obj"
                 scale="${mesh_scale}"/>
         </geometry>
@@ -22,5 +22,5 @@
         <origin xyz="0 0 0" rpy="0 0 0"/>
         <geometry>
-          <mesh filename="${mesh_path}/lap-rf.obj"
+          <mesh filename="package://robot/meshes/lap-rf.obj"
                 scale="${mesh_scale}"/>
         </geometry>

File: src/robot/urdf/motor.xacro (robot description, xacro)
@@ -20,5 +20,5 @@
         <origin xyz="0 0 0" rpy="0 0 0"/>
         <geometry>
-          <mesh filename="${mesh_path}/motor-rf.obj"
+          <mesh filename="package://robot/meshes/motor-rf.obj"
                 scale="${mesh_scale}"/>
         </geometry>
@@ -29,5 +29,5 @@
         <origin xyz="0 0 0" rpy="0 0 0"/>
         <geometry>
-          <mesh filename="${mesh_path}/motor-rf.obj"
+          <mesh filename="package://robot/meshes/motor-rf.obj"
                 scale="${mesh_scale}"/>
         </geometry>

File: src/robot/urdf/radar-front.xacro (robot description, xacro)
@@ -21,5 +21,5 @@
         <origin xyz="0 0 0" rpy="0 0 0"/>
         <geometry>
-          <mesh filename="${mesh_path}/radar-front-rf.obj"
+          <mesh filename="package://robot/meshes/radar-front-rf.obj"
                 scale="${mesh_scale}"/>
         </geometry>
@@ -30,5 +30,5 @@
         <origin xyz="0 0 0" rpy="0 0 0"/>
         <geometry>
-          <mesh filename="${mesh_path}/radar-front-rf.obj"
+          <mesh filename="package://robot/meshes/radar-front-rf.obj"
                 scale="${mesh_scale}"/>
         </geometry>

File: src/robot/urdf/radar-side.xacro (robot description, xacro)
@@ -21,5 +21,5 @@
         <origin xyz="0 0 0" rpy="0 0 0"/>
         <geometry>
-          <mesh filename="${mesh_path}/radar-side-rf.obj"
+          <mesh filename="package://robot/meshes/radar-side-rf.obj"
                 scale="${mesh_scale}"/>
         </geometry>
@@ -30,5 +30,5 @@
         <origin xyz="0 0 0" rpy="0 0 0"/>
         <geometry>
-          <mesh filename="${mesh_path}/radar-side-rf.obj"
+          <mesh filename="package://robot/meshes/radar-side-rf.obj"
                 scale="${mesh_scale}"/>
         </geometry>

File: src/robot/urdf/robot.xacro (robot description, xacro)
@@ -12,6 +12,4 @@
   <!-- 新增：动态获取robot包的绝对路径（核心！） -->
   <xacro:property name="pkg_path" value="$(find robot)"/>
-  <!-- 定义mesh文件夹路径 -->
-  <xacro:property name="mesh_path" value="${pkg_path}/meshes"/>
   <!-- 基础连杆（作为机器人根节点） -->
   <link name="base_link">
@@ -31,5 +29,5 @@
       <origin xyz="0 0 0" rpy="0 0 0"/>
       <geometry>
-        <mesh filename="${mesh_path}/body.obj"
+        <mesh filename="package://robot/meshes/body.obj"
               scale="0.001 0.001 0.001"/>
       </geometry>
@@ -40,5 +38,5 @@
       <origin xyz="0 0 0" rpy="0 0 0"/>
       <geometry>
-        <mesh filename="${mesh_path}/body.obj"
+        <mesh filename="package://robot/meshes/body.obj"
               scale="0.001 0.001 0.001"/>
       </geometry>

File: src/robot/urdf/shin.xacro (robot description, xacro)
@@ -20,5 +20,5 @@
         <origin xyz="0 0 0" rpy="0 0 0"/>
         <geometry>
-          <mesh filename="${mesh_path}/shin-rf.obj"
+          <mesh filename="package://robot/meshes/shin-rf.obj"
                 scale="${mesh_scale}"/>
         </geometry>
@@ -28,5 +28,5 @@
         <origin xyz="0 0 0" rpy="0 0 0"/>
         <geometry>
-          <mesh filename="${mesh_path}/shin-rf.obj"
+          <mesh filename="package://robot/meshes/shin-rf.obj"
                 scale="${mesh_scale}"/>
         </geometry>

File: src/robot/urdf/wheel.xacro (robot description, xacro)
@@ -20,5 +20,5 @@
         <origin xyz="0 0 0" rpy="0 0 0"/>
         <geometry>
-          <mesh filename="${mesh_path}/wheel-rf.obj"
+          <mesh filename="package://robot/meshes/wheel-rf.obj"
                 scale="${mesh_scale}"/>
         </geometry>
@@ -29,5 +29,5 @@
         <origin xyz="0 0 0" rpy="0 0 0"/>
         <geometry>
-          <mesh filename="${mesh_path}/wheel-rf.obj"
+          <mesh filename="package://robot/meshes/wheel-rf.obj"
                 scale="${mesh_scale}"/>
         </geometry>
