Commit message: 底盘控制3种模式通过ros param切换

File: src/robot/urdf/motor.xacro (robot description, xacro)
@@ -47,5 +47,5 @@
       <child link="motor_${suffix}"/>
       <!-- 假设转向绕 Z 轴，根据实际模型可调整为其他轴 -->
-      <axis xyz="0 0 -1"/>
+      <axis xyz="0 0 1"/>
       <!-- 运动范围：-90° 到 90°（-1.57 到 1.57 弧度） -->
       <limit lower="-1.57" upper="1.57" effort="5.0" velocity="1.0"/>

File: src/robot/urdf/robot.xacro (robot description, xacro)
@@ -53,5 +53,5 @@
   <!-- 底盘与身体的固定关节（保留） -->
   <joint name="base_body_joint" type="fixed">
-    <origin xyz="0 0 0" rpy="0 0 0"/>
+    <origin xyz="0 0 0" rpy="0 0 ${pi/2}"/>
     <parent link="base_link"/>
     <child link="body"/>
