Commit message: 双目摄像头标定

File: src/robot/urdf/robot.xacro (robot description, xacro)
@@ -212,5 +212,5 @@
   <!-- 双目安装位姿尚未实测；正式实机导航前必须替换 xyz/rpy。 -->
   <xacro:stereo_camera parent_link="base_link" xyz="0.20 0 0.30"
-                       rpy="0 0 0" baseline="0.065"/>
+                       rpy="0 0 0" baseline="0.061145213"/>
   <xacro:include filename="hardware.xacro"/>
 </robot>

File: src/robot/urdf/stereo_camera.xacro (robot description, xacro)
@@ -2,8 +2,8 @@
 <robot xmlns:xacro="http://www.ros.org/wiki/xacro">
   <!--
-    这里只提供待实测的初始安装位姿和标称 65 mm 几何外观。
-    深度计算必须使用标定 YAML 中的真实投影矩阵，不能使用该标称值。
+    安装位姿仍待实测；默认基线来自 USB Camera 01.00.00 的双目标定结果。
+    深度计算使用标定 YAML 中的投影矩阵，几何基线仅用于同步模型中的镜头位置。
   -->
-  <xacro:macro name="stereo_camera" params="parent_link xyz rpy baseline:=0.065">
+  <xacro:macro name="stereo_camera" params="parent_link xyz rpy baseline:=0.061145213">
     <link name="stereo_camera_link">
       <visual>

Commit message: 增加头部和双目摄像头urdf部分

File: src/robot/urdf/robot.xacro (robot description, xacro)
@@ -11,4 +11,5 @@
   <xacro:include filename="imu.xacro"/>
   <xacro:include filename="stereo_camera.xacro"/>
+  <xacro:include filename="head.xacro"/>
   <!-- 新增：动态获取robot包的绝对路径（核心！） -->
   <xacro:property name="pkg_path" value="$(find robot)"/>
@@ -210,7 +211,20 @@
     yaw="0"
   />
-  <!-- 双目安装位姿尚未实测；正式实机导航前必须替换 xyz/rpy。 -->
-  <xacro:stereo_camera parent_link="base_link" xyz="0.20 0 0.30"
-                       rpy="0 0 0" baseline="0.061145213"/>
+  <!--
+    两自由度头部安装在 body 前方中线。当前位姿依据参考图和网格边界设置，
+    实机装配完成后应测量安装面并校准 xyz/rpy。
+  -->
+  <xacro:head parent_link="body"
+              xyz="0 -0.145 0.205"
+              rpy="0 0 0"
+              mesh_scale="0.001 0.001 0.001"/>
+  <!--
+    双目摄像头安装在头部上半部分内部；两个 OBJ 共享局部装配原点，
+    相机镜头中心与面罩的左右孔重合。
+  -->
+  <xacro:stereo_camera parent_link="head_pitch_link"
+                       xyz="0 0 0"
+                       rpy="0 0 0"
+                       baseline="0.061145213"/>
   <xacro:include filename="hardware.xacro"/>
 </robot>

File: src/robot/urdf/stereo_camera.xacro (robot description, xacro)
@@ -2,17 +2,38 @@
 <robot xmlns:xacro="http://www.ros.org/wiki/xacro">
   <!--
-    安装位姿仍待实测；默认基线来自 USB Camera 01.00.00 的双目标定结果。
-    深度计算使用标定 YAML 中的投影矩阵，几何基线仅用于同步模型中的镜头位置。
+    双目摄像头 OBJ 与 head_pitch_link 使用相同的装配坐标原点。
+    网格镜头中心为 x=±30.5 mm、y=-16.5 mm、z=46.8 mm，孔距为 61 mm。
+    optical frame 继续使用 USB Camera 01.00.00 标定得到的精确基线。
   -->
-  <xacro:macro name="stereo_camera" params="parent_link xyz rpy baseline:=0.061145213">
+  <xacro:macro name="stereo_camera"
+               params="parent_link
+                       xyz:='0 0 0'
+                       rpy:='0 0 0'
+                       baseline:=0.061145213
+                       mesh_scale:='0.001 0.001 0.001'
+                       lens_y:=-0.0165
+                       lens_z:=0.0468">
     <link name="stereo_camera_link">
       <visual>
+        <origin xyz="0 0 0" rpy="0 0 0"/>
         <geometry>
-          <box size="0.09 0.08 0.035"/>
+          <mesh filename="package://robot/meshes/stereo_camera.obj"
+                scale="${mesh_scale}"/>
         </geometry>
-        <material name="stereo_camera_black">
-          <color rgba="0.08 0.08 0.08 1.0"/>
-        </material>
+        <xacro:get_material_by_name material_name="pla_gray_light"/>
       </visual>
+      <collision>
+        <origin xyz="0 0 0" rpy="0 0 0"/>
+        <geometry>
+          <mesh filename="package://robot/meshes/stereo_camera.obj"
+                scale="${mesh_scale}"/>
+        </geometry>
+      </collision>
+      <inertial>
+        <origin xyz="0 -0.0085 0.0468" rpy="0 0 0"/>
+        <mass value="0.08"/>
+        <inertia ixx="0.000015" ixy="0.0" ixz="0.0"
+                 iyy="0.000045" iyz="0.0" izz="0.000050"/>
+      </inertial>
     </link>
     <joint name="stereo_camera_joint" type="fixed">
@@ -21,9 +42,11 @@
       <origin xyz="${xyz}" rpy="${rpy}"/>
     </joint>
+    <!-- 头部局部 +X 为车体左侧，两个镜头沿 X 轴排列并朝向车头 -Y。 -->
     <link name="stereo_left_camera_frame"/>
     <joint name="stereo_left_camera_joint" type="fixed">
       <parent link="stereo_camera_link"/>
       <child link="stereo_left_camera_frame"/>
-      <origin xyz="0 ${baseline / 2.0} 0" rpy="0 0 0"/>
+      <origin xyz="${baseline / 2.0} ${lens_y} ${lens_z}"
+              rpy="0 0 ${-pi / 2.0}"/>
     </joint>
     <link name="stereo_left_optical_frame"/>
@@ -37,5 +60,6 @@
       <parent link="stereo_camera_link"/>
       <child link="stereo_right_camera_frame"/>
-      <origin xyz="0 ${-baseline / 2.0} 0" rpy="0 0 0"/>
+      <origin xyz="${-baseline / 2.0} ${lens_y} ${lens_z}"
+              rpy="0 0 ${-pi / 2.0}"/>
     </joint>
     <link name="stereo_right_optical_frame"/>
