Commit message: 实时建图修改

File: src/robot_description/urdf/hardware.xacro (robot description, xacro)
@@ -77,4 +77,13 @@
       <state_interface name="velocity"/>
     </joint>
+    <!-- 头部几何仍由 head.xacro 定义；此处只提供 ros2_control 位置接口。 -->
+    <joint name="head_yaw_joint">
+      <command_interface name="position"/>
+      <state_interface name="position"/>
+    </joint>
+    <joint name="head_pitch_joint">
+      <command_interface name="position"/>
+      <state_interface name="position"/>
+    </joint>
   </ros2_control>
 </robot>

Commit message: 1.ros2接入实机底盘系统 2.根据ros package增加多agent，处理不同包的内容

File: src/robot_description/urdf/hardware.xacro (robot description, xacro)
@@ -2,8 +2,20 @@
 <!-- 使用方法：由 robot_description/urdf/robot.xacro 组合，通常不要单独启动。 -->
 <robot name="robot_hardware" xmlns:xacro="http://www.ros.org/wiki/xacro">
+  <xacro:macro name="hardware" params="hardware_plugin servo_calibration_file device_candidates serial_timeout_ms inter_command_delay_ms discovery_retry_count discovery_retry_delay_ms encoder_query_delay_ms command_timeout_ms wheel_diameter sonar_lpf_alpha sonar_min_valid_mm sonar_max_valid_mm">
   <ros2_control name="RobotHardware" type="system">
     <hardware>
-      <!-- 🔥 官方自带插件，无需安装任何依赖！ -->
-      <plugin>mock_components/GenericSystem</plugin>
+      <plugin>${hardware_plugin}</plugin>
+      <param name="device_candidates">${device_candidates}</param>
+      <param name="serial_timeout_ms">${serial_timeout_ms}</param>
+      <param name="inter_command_delay_ms">${inter_command_delay_ms}</param>
+      <param name="discovery_retry_count">${discovery_retry_count}</param>
+      <param name="discovery_retry_delay_ms">${discovery_retry_delay_ms}</param>
+      <param name="encoder_query_delay_ms">${encoder_query_delay_ms}</param>
+      <param name="command_timeout_ms">${command_timeout_ms}</param>
+      <param name="wheel_diameter">${wheel_diameter}</param>
+      <param name="sonar_lpf_alpha">${sonar_lpf_alpha}</param>
+      <param name="sonar_min_valid_mm">${sonar_min_valid_mm}</param>
+      <param name="sonar_max_valid_mm">${sonar_max_valid_mm}</param>
+      <param name="servo_calibration_file">${servo_calibration_file}</param>
     </hardware>
     <joint name="lap_body_joint_fr">
@@ -20,20 +32,4 @@
     </joint>
     <joint name="lap_body_joint_rl">
-      <command_interface name="position"/>
-      <state_interface name="position"/>
-    </joint>
-    <joint name="shin_lap_fr_joint_fr">
-      <command_interface name="position"/>
-      <state_interface name="position"/>
-    </joint>
-    <joint name="shin_lap_fl_joint_fl">
-      <command_interface name="position"/>
-      <state_interface name="position"/>
-    </joint>
-    <joint name="shin_lap_rr_joint_rr">
-      <command_interface name="position"/>
-      <state_interface name="position"/>
-    </joint>
-    <joint name="shin_lap_rl_joint_rl">
       <command_interface name="position"/>
       <state_interface name="position"/>
@@ -87,3 +83,4 @@
     </joint>
   </ros2_control>
+  </xacro:macro>
 </robot>

File: src/robot_description/urdf/head.xacro (robot description, xacro)
@@ -70,5 +70,5 @@
       </inertial>
     </link>
-    <!-- pitch 初始限制为上下各 45 度，后续可按实机舵机限位校准。 -->
+    <!-- pitch 按旧控制程序的实机机械限制固定为上下各 30 度。 -->
     <joint name="head_pitch_joint" type="revolute">
       <origin xyz="${pitch_joint_xyz}" rpy="0 0 0"/>
@@ -76,5 +76,5 @@
       <child link="head_pitch_link"/>
       <axis xyz="1 0 0"/>
-      <limit lower="${-pi / 4.0}" upper="${pi / 4.0}"
+      <limit lower="${-pi / 6.0}" upper="${pi / 6.0}"
              effort="3.0" velocity="1.0"/>
       <dynamics damping="0.05" friction="0.0"/>

File: src/robot_description/urdf/lap.xacro (robot description, xacro)
@@ -4,5 +4,5 @@
   <!-- 大腿模块的XACRO宏定义 -->
   <xacro:macro name="lap"
-               params="suffix parent_link
+               params="suffix parent_link lower:='-0.785398' upper:='0.785398'
                        xyz:='0 0 0'
                        rpy:='0 0 0'
@@ -56,5 +56,5 @@
         - velocity: 最大角速度，单位：弧度/秒(rad/s)
       -->
-      <limit lower="${-pi/4}" upper="${pi/4}" effort="10.0" velocity="1.0"/>
+      <limit lower="${lower}" upper="${upper}" effort="10.0" velocity="1.0"/>
       <!--
         dynamics 标签：关节动态特性

File: src/robot_description/urdf/robot.xacro (robot description, xacro)
@@ -2,4 +2,18 @@
 <!-- 使用方法：由 robot_description/description.launch.py 展开并发布完整机器人模型。 -->
 <robot name="robot" xmlns:xacro="http://www.ros.org/wiki/xacro">
+  <!-- mode 只决定 ros2_control 插件；模型、关节和控制接口保持完全一致。 -->
+  <xacro:arg name="hardware_plugin" default="mock_components/GenericSystem"/>
+  <xacro:arg name="servo_calibration_file" default=""/>
+  <xacro:arg name="device_candidates" default="/dev/ttyACM0,/dev/ttyACM1,/dev/ttyACM2"/>
+  <xacro:arg name="serial_timeout_ms" default="500"/>
+  <xacro:arg name="inter_command_delay_ms" default="3"/>
+  <xacro:arg name="discovery_retry_count" default="20"/>
+  <xacro:arg name="discovery_retry_delay_ms" default="700"/>
+  <xacro:arg name="encoder_query_delay_ms" default="20"/>
+  <xacro:arg name="command_timeout_ms" default="500"/>
+  <xacro:arg name="wheel_diameter" default="0.110"/>
+  <xacro:arg name="sonar_lpf_alpha" default="0.2"/>
+  <xacro:arg name="sonar_min_valid_mm" default="30"/>
+  <xacro:arg name="sonar_max_valid_mm" default="2500"/>
   <!-- 引入xacro文件 -->
   <xacro:include filename="materials.xacro"/>
@@ -10,7 +24,9 @@
   <xacro:include filename="radar-front.xacro"/>
   <xacro:include filename="radar-side.xacro"/>
+  <xacro:include filename="sonar.xacro"/>
   <xacro:include filename="imu.xacro"/>
   <xacro:include filename="stereo_camera.xacro"/>
   <xacro:include filename="head.xacro"/>
+  <xacro:include filename="hardware.xacro"/>
   <!-- 新增：动态获取robot包的绝对路径（核心！） -->
   <xacro:property name="pkg_path" value="$(find robot_description)"/>
@@ -64,4 +80,5 @@
   <xacro:lap suffix="fr"
              parent_link="body"
+             lower="${-pi/6}" upper="${pi/4}"
              xyz="-0.091 -0.072 0.158"
              rpy="0 0 0"
@@ -70,4 +87,5 @@
   <xacro:lap suffix="fl"
              parent_link="body"
+             lower="${-pi/4}" upper="${pi/6}"
              xyz="0.091 -0.072 0.158"
              rpy="0 0 0"
@@ -76,4 +94,5 @@
   <xacro:lap suffix="rr"
              parent_link="body"
+             lower="${-pi/4}" upper="${pi/6}"
              xyz="-0.091 0.072 0.158"
              rpy="0 0 0"
@@ -82,4 +101,5 @@
   <xacro:lap suffix="rl"
              parent_link="body"
+             lower="${-pi/6}" upper="${pi/4}"
              xyz="0.091 0.072 0.158"
              rpy="0 0 0"
@@ -89,4 +109,5 @@
   <xacro:shin suffix="fr"
               parent_link="lap_fr"
+              mimic_joint="lap_body_joint_fr"
               xyz="-0.017 -0.060 0"
               rpy="0 0 0"
@@ -95,4 +116,5 @@
   <xacro:shin suffix="fl"
               parent_link="lap_fl"
+              mimic_joint="lap_body_joint_fl"
               xyz="0.017 -0.060 0"
               rpy="0 0 0"
@@ -101,4 +123,5 @@
   <xacro:shin suffix="rr"
               parent_link="lap_rr"
+              mimic_joint="lap_body_joint_rr"
               xyz="-0.017 0.060 0"
               rpy="0 0 0"
@@ -107,4 +130,5 @@
   <xacro:shin suffix="rl"
               parent_link="lap_rl"
+              mimic_joint="lap_body_joint_rl"
               xyz="0.017 0.060 0"
               rpy="0 0 0"
@@ -202,4 +226,13 @@
               rpy="0 0 0"
               mesh_scale="-0.001 -0.001 0.001"/>
+  <!-- 实机固定超声波：前3、后3、左1、右1，位置来自 hw_ctrl/chassis.json。 -->
+  <xacro:sonar_frame name="sonar_fl" parent="base_link" xyz="0.201 0.058 0.03" yaw="${pi/6}"/>
+  <xacro:sonar_frame name="sonar_fc" parent="base_link" xyz="0.215 0 0.03" yaw="0"/>
+  <xacro:sonar_frame name="sonar_fr" parent="base_link" xyz="0.201 -0.058 0.03" yaw="${-pi/6}"/>
+  <xacro:sonar_frame name="sonar_right" parent="base_link" xyz="0 -0.142 0.03" yaw="${-pi/2}"/>
+  <xacro:sonar_frame name="sonar_rr" parent="base_link" xyz="-0.190 -0.062 0.03" yaw="${-2*pi/3}"/>
+  <xacro:sonar_frame name="sonar_rc" parent="base_link" xyz="-0.200 0 0.03" yaw="${pi}"/>
+  <xacro:sonar_frame name="sonar_rl" parent="base_link" xyz="-0.190 0.062 0.03" yaw="${2*pi/3}"/>
+  <xacro:sonar_frame name="sonar_left" parent="base_link" xyz="0 0.142 0.03" yaw="${pi/2}"/>
   <!--  插入 IMU（修改安装位置即可） -->
   <xacro:imu
@@ -228,4 +261,16 @@
                        rpy="0 0 0"
                        baseline="0.061145213"/>
-  <xacro:include filename="hardware.xacro"/>
+  <xacro:hardware hardware_plugin="$(arg hardware_plugin)"
+                  servo_calibration_file="$(arg servo_calibration_file)"
+                  device_candidates="$(arg device_candidates)"
+                  serial_timeout_ms="$(arg serial_timeout_ms)"
+                  inter_command_delay_ms="$(arg inter_command_delay_ms)"
+                  discovery_retry_count="$(arg discovery_retry_count)"
+                  discovery_retry_delay_ms="$(arg discovery_retry_delay_ms)"
+                  encoder_query_delay_ms="$(arg encoder_query_delay_ms)"
+                  command_timeout_ms="$(arg command_timeout_ms)"
+                  wheel_diameter="$(arg wheel_diameter)"
+                  sonar_lpf_alpha="$(arg sonar_lpf_alpha)"
+                  sonar_min_valid_mm="$(arg sonar_min_valid_mm)"
+                  sonar_max_valid_mm="$(arg sonar_max_valid_mm)"/>
 </robot>

File: src/robot_description/urdf/shin.xacro (robot description, xacro)
@@ -12,5 +12,5 @@
   -->
   <xacro:macro name="shin"
-               params="suffix parent_link
+               params="suffix parent_link mimic_joint
                        xyz:='0 0 0'
                        rpy:='0 0 0'
@@ -48,4 +48,6 @@
       <!-- 假设膝盖绕 X 轴旋转，请根据实际模型调整 -->
       <axis xyz="1 0 0"/>
+      <!-- 实机每条腿只有一个主动轴，小腿通过连杆反向补偿大腿角度。 -->
+      <mimic joint="${mimic_joint}" multiplier="-1.0" offset="0.0"/>
       <limit lower="-0.785" upper="0.785" effort="5.0" velocity="1.0"/>
       <dynamics damping="0.05" friction="0.0"/>

Commit message: 接入实机底盘系统后测试轮子、大腿已完成

File: src/robot_description/urdf/hardware.xacro (robot description, xacro)
@@ -2,5 +2,5 @@
 <!-- 使用方法：由 robot_description/urdf/robot.xacro 组合，通常不要单独启动。 -->
 <robot name="robot_hardware" xmlns:xacro="http://www.ros.org/wiki/xacro">
-  <xacro:macro name="hardware" params="hardware_plugin servo_calibration_file device_candidates serial_timeout_ms inter_command_delay_ms discovery_retry_count discovery_retry_delay_ms encoder_query_delay_ms command_timeout_ms wheel_diameter sonar_lpf_alpha sonar_min_valid_mm sonar_max_valid_mm">
+  <xacro:macro name="hardware" params="hardware_plugin servo_calibration_file wheel_calibration_file device_candidates serial_timeout_ms inter_command_delay_ms discovery_retry_count discovery_retry_delay_ms encoder_query_delay_ms command_timeout_ms wheel_diameter sonar_lpf_alpha sonar_min_valid_mm sonar_max_valid_mm">
   <ros2_control name="RobotHardware" type="system">
     <hardware>
@@ -18,4 +18,5 @@
       <param name="sonar_max_valid_mm">${sonar_max_valid_mm}</param>
       <param name="servo_calibration_file">${servo_calibration_file}</param>
+      <param name="wheel_calibration_file">${wheel_calibration_file}</param>
     </hardware>
     <joint name="lap_body_joint_fr">

File: src/robot_description/urdf/robot.xacro (robot description, xacro)
@@ -5,4 +5,5 @@
   <xacro:arg name="hardware_plugin" default="mock_components/GenericSystem"/>
   <xacro:arg name="servo_calibration_file" default=""/>
+  <xacro:arg name="wheel_calibration_file" default=""/>
   <xacro:arg name="device_candidates" default="/dev/ttyACM0,/dev/ttyACM1,/dev/ttyACM2"/>
   <xacro:arg name="serial_timeout_ms" default="500"/>
@@ -80,5 +81,5 @@
   <xacro:lap suffix="fr"
              parent_link="body"
-             lower="${-pi/6}" upper="${pi/4}"
+             lower="${-pi/6}" upper="${pi/6}"
              xyz="-0.091 -0.072 0.158"
              rpy="0 0 0"
@@ -87,5 +88,5 @@
   <xacro:lap suffix="fl"
              parent_link="body"
-             lower="${-pi/4}" upper="${pi/6}"
+             lower="${-pi/6}" upper="${pi/6}"
              xyz="0.091 -0.072 0.158"
              rpy="0 0 0"
@@ -94,5 +95,5 @@
   <xacro:lap suffix="rr"
              parent_link="body"
-             lower="${-pi/4}" upper="${pi/6}"
+             lower="${-pi/6}" upper="${pi/6}"
              xyz="-0.091 0.072 0.158"
              rpy="0 0 0"
@@ -101,5 +102,5 @@
   <xacro:lap suffix="rl"
              parent_link="body"
-             lower="${-pi/6}" upper="${pi/4}"
+             lower="${-pi/6}" upper="${pi/6}"
              xyz="0.091 0.072 0.158"
              rpy="0 0 0"
@@ -263,4 +264,5 @@
   <xacro:hardware hardware_plugin="$(arg hardware_plugin)"
                   servo_calibration_file="$(arg servo_calibration_file)"
+                  wheel_calibration_file="$(arg wheel_calibration_file)"
                   device_candidates="$(arg device_candidates)"
                   serial_timeout_ms="$(arg serial_timeout_ms)"
