Commit message: 机器人启动launch文件优化，网页优化，超声波增加有效距离过滤

File: ROS2/src/robot_description/urdf/hardware.xacro (robot description, xacro)
@@ -2,5 +2,5 @@
 <!-- 使用方法：由 robot_description/urdf/robot.xacro 组合，通常不要单独启动。 -->
 <robot name="robot_hardware" xmlns:xacro="http://www.ros.org/wiki/xacro">
-  <xacro:macro name="hardware" params="hardware_plugin servo_calibration_file wheel_calibration_file device_candidates serial_timeout_ms inter_command_delay_ms discovery_retry_count discovery_retry_delay_ms encoder_query_delay_ms command_timeout_ms wheel_diameter sonar_lpf_alpha sonar_min_valid_mm sonar_max_valid_mm">
+  <xacro:macro name="hardware" params="hardware_plugin servo_calibration_file wheel_calibration_file device_candidates serial_timeout_ms inter_command_delay_ms discovery_retry_count discovery_retry_delay_ms encoder_query_delay_ms command_timeout_ms servo_keepalive_period_ms servo_command_timeout_ms wheel_diameter sonar_lpf_alpha sonar_min_valid_mm sonar_max_valid_mm">
   <ros2_control name="RobotHardware" type="system">
     <hardware>
@@ -13,4 +13,6 @@
       <param name="encoder_query_delay_ms">${encoder_query_delay_ms}</param>
       <param name="command_timeout_ms">${command_timeout_ms}</param>
+      <param name="servo_keepalive_period_ms">${servo_keepalive_period_ms}</param>
+      <param name="servo_command_timeout_ms">${servo_command_timeout_ms}</param>
       <param name="wheel_diameter">${wheel_diameter}</param>
       <param name="sonar_lpf_alpha">${sonar_lpf_alpha}</param>

File: ROS2/src/robot_description/urdf/robot.xacro (robot description, xacro)
@@ -13,4 +13,6 @@
   <xacro:arg name="encoder_query_delay_ms" default="20"/>
   <xacro:arg name="command_timeout_ms" default="500"/>
+  <xacro:arg name="servo_keepalive_period_ms" default="40"/>
+  <xacro:arg name="servo_command_timeout_ms" default="400"/>
   <xacro:arg name="wheel_diameter" default="0.110"/>
   <xacro:arg name="sonar_lpf_alpha" default="0.2"/>
@@ -272,4 +274,6 @@
                   encoder_query_delay_ms="$(arg encoder_query_delay_ms)"
                   command_timeout_ms="$(arg command_timeout_ms)"
+                  servo_keepalive_period_ms="$(arg servo_keepalive_period_ms)"
+                  servo_command_timeout_ms="$(arg servo_command_timeout_ms)"
                   wheel_diameter="$(arg wheel_diameter)"
                   sonar_lpf_alpha="$(arg sonar_lpf_alpha)"
